File: HB-RC-12-EP-2.kicad_pcb (KiCad board)
At the start: 2 copper layers, 48 x 89.5 mm, 69 parts, among them J3 eInk, K1 ePaper, Q1 CSTCE8, Q2 IRLML6346TRBPF, Q3 CSTCC8, SW1 SW_Push, SW10 SW_Push, SW11 SW_Push, SW12 SW_Push, SW2 SW_Push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

Commit message: Bugfix
Parts:
- moved D1 0.08 mm to (134.1, 75.3)
- moved D2 0.08 mm to (132.2, 75.3)
- moved D6 0.05 mm to (130.2, 75.3)
Routing:
- net GND: track 99.3 -> 99.9 mm
Other:
- outline, holes or cut-outs redrawn
- board text added: "HB-RC-12-EP PCB V2.0 maxx3105"
- board text added: "RESET"
- board text removed: "RESEt"
